File: 8probe/Probe Board 1.0.sch (EAGLE design)
At the start: 61 parts, among them Q3 2N7002, Q4 2N7002, U1 LTC2495CUHFPBF, U3 MAX6037AAUKADJ+T, U4 CSTCE16M0V53A-R0, U5 TPS79733DCKR, U6 ATMEGA328P_TQFPQFN_32

Commit message: Minor layout updates to 8probe
Split ground plane redistributed decoupling capacitors appropriately, moved input cable connections to be in a row, fixed package on Q1 and Q2, corrected ground pad on ATMEGA. Silk screen still needs updating
Parts:
- removed Q3, Q4: 2N7002, 2N7002(2):2N7002
- removed R18: 30k, SparkFun:RESISTOR0603-RES
- added Q1, Q2: 2N7002, bschulz:MOSFET-NCH-2N7002PW
Connections:
- removed net N$9: R18.2, U5.PG
- net 3.3V: now also Q1.G, Q2.G; no longer Q3.1, Q4.1, R18.1
- net SCL3.3V: now also Q2.S; no longer Q3.3
- net SCL5V: now also Q2.D; no longer Q3.2
- net SDA3.3V: now also Q1.S; no longer Q4.3
- net SDA5V: now also Q1.D; no longer Q4.2
Other:
- moved on the sheet: U6
Changed lines of the file:
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@@
 <?xml version="1.0" encoding="utf-8"?>
 <!DOCTYPE eagle SYSTEM "eagle.dtd">
-<eagle version="9.3.0">
+<eagle version="9.2.1">
 <drawing>
 <settings>
@@
 <part name="P+2" library="SparkFun" deviceset="3.3V" device=""/>
 <part name="U$18" library="MyPOW" deviceset="+5V" device=""/>
-<part name="Q3" library="2N7002(2)" deviceset="2N7002" device="">
-<attribute name="DIGIKEY_PART_NUMBER" value="2N7002NCT-ND"/>
-<attribute name="MANUFACTURER" value="ON Semiconductor"/>
-<attribute name="PRICE" value="0.06193"/>
-<attribute name="VENDOR" value="ON Semiconductor"/>
-</part>
-<part name="Q4" library="2N7002(2)" deviceset="2N7002" device="">
-<attribute name="DIGIKEY_PART_NUMBER" value="2N7002NCT-ND"/>
-<attribute name="MANUFACTURER" value="ON Semiconductor"/>
-<attribute name="PRICE" value="0.06193"/>
-</part>
 <part name="U5" library="TPS79733" deviceset="TPS79733DCKR" device="">
 <attribute name="DIGIKEY_PART_NUMBER" value="296-11990-6-ND"/>
@@
 <part name="U$41" library="MyPOW" deviceset="COM" device=""/>
 <part name="U$42" library="MyPOW" deviceset="COM" device=""/>
-<part name="R18" library="SparkFun" deviceset="RESISTOR" device="0603-RES" value="30k">
-<attribute name="DIGIKEY_PART_NUMBER" value="P30KGDKR-ND"/>
-<attribute name="MANUFACTURER" value="Panasonic Electronic Components"/>
-<attribute name="MANUFACTURER_PART_NUMBER" value="ERJ-3GEYJ303V"/>
-<attribute name="PRICE" value="0.00758"/>
-</part>
-<part name="P+5" library="SparkFun" deviceset="3.3V" device=""/>
 <part name="U4" library="Murata Resonator" deviceset="CSTCE16M0V53A-R0" device="">
 <attribute name="DIGIKEY_PART_NUMBER" value="490-1198-1-ND"/>
@@
 <part name="U$45" library="MyPOW" deviceset="COM" device=""/>
 <part name="U$46" library="Smartprj" deviceset="MYPOW_+5V" device="" value="+5V"/>
+<part name="Q1" library="bschulz" deviceset="MOSFET-NCH" device="-2N7002PW" value="2N7002"/>
+<part name="Q2" library="bschulz" deviceset="MOSFET-NCH" device="-2N7002PW" value="2N7002"/>
 </parts>
 <sheets>
@@
 <attribute name="VALUE" x="-132.08" y="124.46" size="1.778" layer="96"/>
 </instance>
-<instance part="Q3" gate="A" x="-142.24" y="147.32" smashed="yes" rot="R270">
-<attribute name="DIGIKEY_PART_NUMBER" x="-142.24" y="147.32" size="1.778" layer="96" rot="R270" display="off"/>
-<attribute name="MANUFACTURER" x="-142.24" y="147.32" size="1.778" layer="96" rot="R270" display="off"/>
-<attribute name="PRICE" x="-142.24" y="147.32" size="1.778" layer="96" rot="R270" display="off"/>
-<attribute name="NAME" x="-141.605" y="135.89" size="2.54" layer="95" ratio="10" rot="SR270"/>
-<attribute name="VALUE" x="-146.05" y="135.89" size="2.54" layer="96" ratio="10" rot="SR270"/>
-</instance>
-<instance part="Q4" gate="A" x="-142.24" y="109.22" smashed="yes" rot="R270">
-<attribute name="DIGIKEY_PART_NUMBER" x="-142.24" y="109.22" size="1.778" layer="96" rot="R270" display="off"/>
-<attribute name="MANUFACTURER" x="-142.24" y="109.22" size="1.778" layer="96" rot="R270" display="off"/>
-<attribute name="PRICE" x="-142.24" y="109.22" size="1.778" layer="96" rot="R270" display="off"/>
-<attribute name="NAME" x="-141.605" y="97.79" size="2.54" layer="95" ratio="10" rot="SR270"/>
-<attribute name="VALUE" x="-146.05" y="97.79" size="2.54" layer="96" ratio="10" rot="SR270"/>
-</instance>
 <instance part="U5" gate="A" x="-121.92" y="50.8" smashed="yes">
 <attribute name="DIGIKEY_PART_NUMBER" x="-121.92" y="50.8" size="1.778" layer="96" display="off"/>
@@
 <instance part="U$41" gate="G$1" x="-93.98" y="33.02" smashed="yes"/>
 <instance part="U$42" gate="G$1" x="-60.96" y="68.58" smashed="yes" rot="R180"/>
-<instance part="R18" gate="G$1" x="-127" y="50.8" smashed="yes">
-<attribute name="DIGIKEY_PART_NUMBER" x="-127" y="50.8" size="1.778" layer="96" display="off"/>
-<attribute name="MANUFACTURER" x="-127" y="50.8" size="1.778" layer="96" display="off"/>
-<attribute name="MANUFACTURER_PART_NUMBER" x="-127" y="50.8" size="1.778" layer="96" display="off"/>
-<attribute name="PRICE" x="-127" y="50.8" size="1.778" layer="96" display="off"/>
-<attribute name="NAME" x="-130.81" y="52.2986" size="1.778" layer="95"/>
-<attribute name="VALUE" x="-130.81" y="47.498" size="1.778" layer="96"/>
-</instance>
-<instance part="P+5" gate="G$1" x="-137.16" y="53.34" smashed="yes">
-<attribute name="VALUE" x="-138.176" y="56.896" size="1.778" layer="96"/>
-</instance>
 <instance part="R16" gate="G$1" x="-101.6" y="142.24" smashed="yes" rot="R270">
 <attribute name="DIGIKEY_PART_NUMBER" x="-101.6" y="142.24" size="1.778" layer="96" rot="R270" display="off"/>
@@
 </instance>
 <instance part="U$36" gate="G$1" x="-101.6" y="111.76" smashed="yes"/>
+<instance part="Q1" gate="NMOS" x="-142.24" y="104.14" smashed="yes" rot="R270">
+<attribute name="NAME" x="-142.24" y="99.06" size="1.778" layer="95" font="vector" rot="R270"/>
+<attribute name="VALUE" x="-144.78" y="99.06" size="1.778" layer="96" font="vector" rot="R270"/>
+</instance>
+<instance part="Q2" gate="NMOS" x="-142.24" y="142.24" smashed="yes" rot="R270">
+<attribute name="NAME" x="-142.24" y="137.16" size="1.778" layer="95" font="vector" rot="R270"/>
+<attribute name="VALUE" x="-144.78" y="137.16" size="1.778" layer="96" font="vector" rot="R270"/>
+</instance>
 </instances>
 <busses>
@@
 <segment>
 <pinref part="R1" gate="G$1" pin="1"/>
-<wire x1="-129.54" y1="144.78" x2="-129.54" y2="140.335" width="0.1524" layer="91"/>
-<wire x1="-129.54" y1="140.335" x2="-137.16" y2="140.335" width="0.1524" layer="91"/>
+<wire x1="-129.54" y1="144.78" x2="-129.54" y2="142.24" width="0.1524" layer="91"/>
 <label x="-129.54" y="142.24" size="1.27" layer="95"/>
-<pinref part="Q3" gate="A" pin="2"/>
+<pinref part="Q2" gate="NMOS" pin="D"/>
+<wire x1="-129.54" y1="142.24" x2="-129.54" y2="140.335" width="0.1524" layer="91"/>
+<wire x1="-137.16" y1="139.7" x2="-129.54" y2="139.7" width="0.1524" layer="91"/>
+<wire x1="-129.54" y1="139.7" x2="-129.54" y2="140.335" width="0.1524" layer="91"/>
 </segment>
 </net>
@@
 <segment>
 <pinref part="R15" gate="G$1" pin="1"/>
-<wire x1="-129.54" y1="106.68" x2="-129.54" y2="102.235" width="0.1524" layer="91"/>
-<wire x1="-129.54" y1="102.235" x2="-137.16" y2="102.235" width="0.1524" layer="91"/>
+<wire x1="-129.54" y1="106.68" x2="-129.54" y2="104.14" width="0.1524" layer="91"/>
 <label x="-129.54" y="104.14" size="1.27" layer="95"/>
-<pinref part="Q4" gate="A" pin="2"/>
+<pinref part="Q1" gate="NMOS" pin="D"/>
+<wire x1="-129.54" y1="104.14" x2="-129.54" y2="102.235" width="0.1524" layer="91"/>
+<wire x1="-137.16" y1="101.6" x2="-129.54" y2="101.6" width="0.1524" layer="91"/>
+<wire x1="-129.54" y1="101.6" x2="-129.54" y2="102.235" width="0.1524" layer="91"/>
 </segment>
 </net>
@@
 <segment>
 <pinref part="R11" gate="G$1" pin="1"/>
-<wire x1="-154.94" y1="106.68" x2="-154.94" y2="102.235" width="0.1524" layer="91"/>
-<wire x1="-154.94" y1="102.235" x2="-147.32" y2="102.235" width="0.1524" layer="91"/>
+<wire x1="-154.94" y1="106.68" x2="-154.94" y2="104.14" width="0.1524" layer="91"/>
 <label x="-154.94" y="104.14" size="1.27" layer="95"/>
-<pinref part="Q4" gate="A" pin="3"/>
+<pinref part="Q1" gate="NMOS" pin="S"/>
+<wire x1="-154.94" y1="104.14" x2="-154.94" y2="102.235" width="0.1524" layer="91"/>
+<wire x1="-147.32" y1="101.6" x2="-154.94" y2="101.6" width="0.1524" layer="91"/>
+<wire x1="-154.94" y1="101.6" x2="-154.94" y2="102.235" width="0.1524" layer="91"/>
 </segment>
 <segment>
@@
 <segment>
 <pinref part="R2" gate="G$1" pin="1"/>
-<wire x1="-154.94" y1="144.78" x2="-154.94" y2="140.335" width="0.1524" layer="91"/>
-<wire x1="-154.94" y1="140.335" x2="-147.32" y2="140.335" width="0.1524" layer="91"/>
+<wire x1="-154.94" y1="144.78" x2="-154.94" y2="142.24" width="0.1524" layer="91"/>
 <label x="-154.94" y="142.24" size="1.27" layer="95"/>
-<pinref part="Q3" gate="A" pin="3"/>
+<pinref part="Q2" gate="NMOS" pin="S"/>
+<wire x1="-154.94" y1="142.24" x2="-154.94" y2="140.335" width="0.1524" layer="91"/>
+<wire x1="-147.32" y1="139.7" x2="-154.94" y2="139.7" width="0.1524" layer="91"/>
+<wire x1="-154.94" y1="139.7" x2="-154.94" y2="140.335" width="0.1524" layer="91"/>
 </segment>
 <segment>
@@
 <wire x1="-154.94" y1="154.94" x2="-154.94" y2="157.48" width="0.1524" layer="91"/>
 <pinref part="P+1" gate="G$1" pin="3.3V"/>
-<wire x1="-142.24" y1="147.32" x2="-142.24" y2="154.94" width="0.1524" layer="91"/>
-<wire x1="-142.24" y1="154.94" x2="-154.94" y2="154.94" width="0.1524" layer="91"/>
 <junction x="-154.94" y="154.94"/>
-<pinref part="Q3" gate="A" pin="1"/>
+<pinref part="Q2" gate="NMOS" pin="G"/>
+<wire x1="-144.78" y1="154.94" x2="-154.94" y2="154.94" width="0.1524" layer="91"/>
+<wire x1="-144.78" y1="147.32" x2="-144.78" y2="154.94" width="0.1524" layer="91"/>
 </segment>
 <segment>
@@
 <pinref part="R11" gate="G$1" pin="2"/>
 <wire x1="-154.94" y1="119.38" x2="-154.94" y2="116.84" width="0.1524" layer="91"/>
-<wire x1="-142.24" y1="109.22" x2="-142.24" y2="116.84" width="0.1524" layer="91"/>
-<wire x1="-142.24" y1="116.84" x2="-154.94" y2="116.84" width="0.1524" layer="91"/>
 <junction x="-154.94" y="116.84"/>
-<pinref part="Q4" gate="A" pin="1"/>
+<pinref part="Q1" gate="NMOS" pin="G"/>
+<wire x1="-144.78" y1="116.84" x2="-154.94" y2="116.84" width="0.1524" layer="91"/>
+<wire x1="-144.78" y1="109.22" x2="-144.78" y2="116.84" width="0.1524" layer="91"/>
 </segment>
 <segment>
@@
 <junction x="-60.96" y="50.8"/>
 </segment>
-<segment>
-<pinref part="P+5" gate="G$1" pin="3.3V"/>
-<wire x1="-137.16" y1="53.34" x2="-137.16" y2="50.8" width="0.1524" layer="91"/>
-<pinref part="R18" gate="G$1" pin="1"/>
-<wire x1="-137.16" y1="50.8" x2="-132.08" y2="50.8" width="0.1524" layer="91"/>
-</segment>
 </net>
 <net name="IO4" class="0">
@@
 </segment>
 </net>
-<net name="N$9" class="0">
-<segment>
-<pinref part="R18" gate="G$1" pin="2"/>
-<pinref part="U5" gate="A" pin="PG"/>
-<wire x1="-121.92" y1="50.8" x2="-119.38" y2="50.8" width="0.1524" layer="91"/>
-</segment>
-</net>
