File: 8probe/ProbeBoard.brd (EAGLE design)
At the start: 54 x 13 mm, 60 parts, among them Q1 2N7002, Q2 2N7002, U1 LTC2495CUHFPBF, U3 MAX6037AAUKADJ+T, U4 CSTCE16M0V53A-R0, U5 TPS79733DCKR, U6 ATMEGA328P_TQFPQFN_32

Commit message: Updates to 8probe layout, 8probe v0.1 to fab
Minor updates and cleanup to 8probe layout, generated gerbers for 8probe v0.1 sent to fab
Parts:
- removed U3: MAX6037AAUKADJ+T, MAX6037AAUKADJ:21-0057F
- removed U4: CSTCE16M0V53A-R0, Murata Resonator:CSTCE_V
- added U2: TPS79733, bschulz:DCK_R-PDSO-G5
- added Y1: 16MHz, bschulz:RESONATOR-SMD-3.2X1.3
- C1, C10, C2, C3, C5, C7, C8, C9: device SparkFun:0603-CAP -> bschulz_passives:C0603
- R1, R10, R11, R12, R13, R14, R15, R19, R2, R20, R3, R4, R5, R6, R7, R8, R9: device SparkFun:0603-RES -> bschulz_passives:R0603
- R16: value 1k -> 10k; device SparkFun:0603-RES -> bschulz_passives:R0603
- R17: value 2.2k -> 30k; device SparkFun:0603-RES -> bschulz_passives:R0603
- U1: value LTC2495CUHFPBF -> LTC2495_LTC2495CUHFPBF; device LTC2495:QFN-38_UHF -> ProbeBoard:LTC2495_QFN-38_UHF
- U5: value TPS79733DCKR -> MAX6037ADJSOT23; device TPS79733:DCK5 -> bschulz:SOT23-5
- moved U5 8.45 mm to (52.3, 2.79)
- moved R7 4.45 mm to (49.5, 2.41)
- moved C8 1.28 mm to (55.2, 2.41)
- moved C7 0.08 mm to (58.6, 6.17), turned to 0 degrees
- turned R5 to 90 degrees
Connections:
- removed net N$6: R5.1, R7.2, U3.1
- new net N$4: R5.1, R7.2, U5.1
- net +5V: now also C7.2, U2.4, U5.3; no longer C7.1, U3.3, U3.4
- net 3.3V: now also U2.5; no longer U5.5
- net COM: now also C7.1, U2.2, Y1.2; no longer C7.2, U3.2, U4.2
- net N$1: now also Y1.3; no longer U4.3
- net N$7: now also Y1.1; no longer U4.1
- net REF_V: now also U5.5; no longer U3.5
- net SCL5V: now also U6.28
- net SDA5V: now also U6.27
Routing:
- net SDA5V: track 26.7 -> 38.8 mm
- net COM: track 30.2 -> 20.4 mm
- net N$6: track 7.21 -> 0.00 mm
- net REF_V: track 29.4 -> 34.0 mm
- net N$4: track 0.00 -> 4.00 mm
- net SCL5V: track 20.5 -> 23.4 mm
- net +5V: track 147.2 -> 145.3 mm
- net N$7: track 2.84 -> 3.37 mm
Other:
- outline, holes or cut-outs redrawn
- board text added: "Thermal Stake-8 v0.1 Evan Grove Bobby Schulz"
- board text added: "VCC"
- board text added: "Vin"
- board text removed: "+5V"
- board text removed: "COM"
- board text removed: "v0.1 (8)"
